File: redox/pcb/rev1.0/kicad_files/redox_rev1.sch (KiCad schematic (older format))
At the start: 76 parts, among them K0 KEYSW, K1 KEYSW, K10 KEYSW, K11 KEYSW, K12 KEYSW, K13 KEYSW, K14 KEYSW, K15 KEYSW, K16 KEYSW, K2 KEYSW, K20 KEYSW, K21 KEYSW, K22 KEYSW, K23 KEYSW, K24 KEYSW, K25 KEYSW, K26 KEYSW, K3 KEYSW, K30 KEYSW, K31 KEYSW, K32 KEYSW, K33 KEYSW, K34 KEYSW, K35 KEYSW, K36 KEYSW, K4 KEYSW, K40 KEYSW, K41 KEYSW, K42 KEYSW, K43 KEYSW, K44 KEYSW, K45 KEYSW, K46 KEYSW, K5 KEYSW, K6 KEYSW, U1 ProMicro

Commit message: added micro and supporting circuitry
Parts:
- removed RGB_STRIP1: Conn_01x03, Pin_Headers:Pin_Header_Straight_1x03_Pitch2.54mm, symbol Conn_01x03
- removed U1: ProMicro, Keebio-Parts:ArduinoProMicro, symbol ProMicro
- added C1: 10n, Capacitor_SMD:C_0805_2012Metric_Pad1.15x1.40mm_HandSolder, symbol Device:C
- added C2: 100n, Capacitor_SMD:C_0805_2012Metric_Pad1.15x1.40mm_HandSolder, symbol Device:C
- added C3: 4,7u, Capacitor_SMD:C_0805_2012Metric_Pad1.15x1.40mm_HandSolder, symbol Device:C
- added C4, C5: 22u, symbol Device:C_Small
- added C6: 100n, symbol Device:C_Small
- added C7: 4.7u, symbol Device:C_Small
- added D1: Schottky, symbol Device:D_Schottky_Small
- added D1: LED, symbol Device:LED_Small
- added FB1: blm18pg221, symbol Device:Ferrite_Bead_Small
- added J1: USB_B_Micro, Connector_USB:USB_Micro-B_Molex-105133-0001, symbol Connector:USB_B_Micro
- added J2: jlink, redox_parts:j-link-6-pin, symbol Connector:Conn_01x06_Female
- added L1: 3.3u, symbol Device:L
- added R1: 100K, Resistor_SMD:R_0805_2012Metric_Pad1.15x1.40mm_HandSolder, symbol Device:R
- added R2: 45K3, symbol Device:R_Small
- added R3: 10K, symbol Device:R_Small
- added R4: 330, symbol Device:R_Small
- added R5: 100K, symbol Device:R_Small
- added U1: STM32F042K6Tx, Package_QFP:LQFP-32_7x7mm_P0.8mm, symbol MCU_ST_STM32F0:STM32F042K6Tx
- added U2: USBLC6-2SC6, Package_TO_SOT_SMD:SOT-23-6, symbol Power_Protection:USBLC6-2SC6
- added U3: LMR10510XMF, Package_TO_SOT_SMD:SOT-23-5, symbol Regulator_Switching:LMR10510XMF
- D0, D1, D10, D11, D12, D13, D14, D15, D16, D2, D20, D21, D22, D23, D24, D25, D26, D3, D30, D31, D32, D33, D34, D35, D36, D4, D40, D41, D42, D43, D44, D45, D46, D5, D6: footprint Keebio-Parts:Diode-dual -> redox_parts:Diode-dual; symbol D -> redox_rev1-rescue:D
- K0, K1, K10, K11, K12, K13, K14, K15, K16, K2, K20, K21, K22, K23, K24, K25, K26, K3, K30, K31, K32, K33, K34, K35, K36, K4, K40, K41, K42, K43, K44, K45, K46, K5, K6: footprint Keebio-Parts:Hybrid_PCB_100H_Dual_hole-nosilk -> redox_parts:Mx_Alps_100-dualside; symbol KEYSW -> redox_rev1-rescue:KEYSW
- R1, R2: symbol R -> redox_rev1-rescue:R
- RST_SW1: footprint Buttons_Switches_ThroughHole:SW_PUSH_6mm_h4.3mm -> redox_parts:SW_PUSH_6mm_h4.3mm; symbol SW_PUSH -> redox_rev1-rescue:SW_PUSH
- TRRS1: footprint Keebio-Parts:TRRS-PJ-320A-dual -> redox_parts:TRRS-PJ-320A-dual; symbol Audio-Jack-4 -> redox_rev1-rescue:Audio-Jack-4
Connections:
- net labels added: +3.3V, +5V, SWCLK, SWDIO, SWO, USB+, USB-, USB_DM, USB_DP, VDD, nRESET
- net labels removed: VCC, rgb_data
- wire segments 69 -> 186
- no-connect marks 4 -> 0

Commit message: schematic checked
Parts:
- removed J2: jlink, redox_parts:j-link-6-pin, symbol Connector:Conn_01x06_Female
- added C8: 0.1u, Capacitor_SMD:C_0805_2012Metric_Pad1.15x1.40mm_HandSolder, symbol Device:C_Small
- added J2: jlink, redox_parts:jlink_10-PIN_NEEDLE_ADAPTER, symbol jlink:8.06.05_10-PIN_NEEDLE_ADAPTER
- C1, C2, C3: symbol Device:C -> Device:C_Small
- C4, C5, C6, C7: footprint (none) -> Capacitor_SMD:C_0805_2012Metric_Pad1.15x1.40mm_HandSolder
- D47: renamed from D1; footprint (none) -> Diode_SMD:D_SOD-123
- D48: renamed from D1; footprint (none) -> Diode_SMD:D_0805_2012Metric_Pad1.15x1.40mm_HandSolder
- FB1: footprint (none) -> Diode_SMD:D_0603_1608Metric_Pad1.05x0.95mm_HandSolder
- L1: footprint (none) -> Inductor_SMD:L_1008_2520Metric
- R1: symbol Device:R -> Device:R_Small
- R2, R3, R4, R5: footprint (none) -> Resistor_SMD:R_0805_2012Metric_Pad1.15x1.40mm_HandSolder
- R6: renamed from R1; footprint Keebio-Parts:Resistor-Compact -> redox_parts:Resistor-Compact
- R7: renamed from R2; footprint Keebio-Parts:Resistor-Compact -> redox_parts:Resistor-Compact
Connections:
- net RST is gone; now on net nRESET: RST_SW1.1
- net +3V3: now also J2.1 (VTREF)
- net GND: now also C8.2, J2.3 (GND)
- net SWCLK: now also J2.4 (SWCLK/TCK)
- net SWDIO: now also J2.2 (SWDIO/TMS)
- net SWO: now also J2.6 (SWO/TDO)
- net nRESET: now also C8.1, J2.10 (NRESET)
Other:
- moved on the sheet: RST_SW1
